File: glr-2024e-bms-can-shield.kicad_pcb (KiCad board)
At the start: 2 copper layers, 70 x 81 mm, 18 parts, among them CN10 Conn_02x19_Odd_Even_MountingP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, CN7 Conn_02x19_Odd_Even_MountingP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, IC1 TLE6250GV33XUMA1, IC2 TLE6250GV33XUMA1, J1 691321100002, J2 691321100004, J3 691321100004, K1 G5V-2, Q1 BC107, Q2 BC107

Commit message: forgor to save the file
add plot output directory

Co-Authored-By: wallalex0 <97884125+wallalex0@users.noreply.github.com>
Parts:
- Q1, Q2: value BC107 -> Q_NPN_EBC
Changed lines of the file:
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@@
 			)
 		)
-		(property "Value" "BC107"
+		(property "Value" "Q_NPN_EBC"
 			(at 0 2.4 90)
 			(layer "F.Fab")
@@
 			)
 		)
-		(property "Datasheet" "http://www.b-kainka.de/Daten/Transistor/BC108.pdf"
+		(property "Datasheet" ""
 			(at 0 0 90)
 			(layer "F.Fab")
@@
 			)
 		)
-		(property "Description" "0.1A Ic, 50V Vce, Low Noise General Purpose NPN Transistor, TO-18"
+		(property "Description" "NPN transistor, emitter/base/collector"
 			(at 0 0 90)
 			(layer "F.Fab")
@@
 			)
 		)
-		(property ki_fp_filters "TO?18*")
 		(sheetname "/")
 		(sheetfile "glr-2024e-bms-can-shield.kicad_sch")
@@
 			)
 		)
-		(property "Value" "BC107"
+		(property "Value" "Q_NPN_EBC"
 			(at 0 2.4 90)
 			(layer "F.Fab")
@@
 			)
 		)
-		(property "Datasheet" "http://www.b-kainka.de/Daten/Transistor/BC108.pdf"
+		(property "Datasheet" ""
 			(at 0 0 90)
 			(layer "F.Fab")
@@
 			)
 		)
-		(property "Description" "0.1A Ic, 50V Vce, Low Noise General Purpose NPN Transistor, TO-18"
+		(property "Description" "NPN transistor, emitter/base/collector"
 			(at 0 0 90)
 			(layer "F.Fab")
@@
 			)
 		)
-		(property ki_fp_filters "TO?18*")
 		(sheetname "/")
 		(sheetfile "glr-2024e-bms-can-shield.kicad_sch")
